File: STM32F042K6Tx.sch (KiCad schematic (older format))
At the start: 9 parts, among them U1 STM32F042K6Tx, X1 ASV-8.000MHz

Commit message: label clkin net
Connections:
- net clkin: now reaches U1.2 (PF0), X1.3 (OUT)
Changed lines of the file:
@@
 	6850 2050 6850 1950
 Connection ~ 6850 1950
+Text Label 3950 3400 0    50   ~ 0
+clkin
 $EndSCHEMATC

Commit message: initial routing mostly finished
Parts:
- NT1: footprint NetTie:NetTie-2_THT_Pad1.0mm -> NetTie:NetTie-2_SMD_Pad0.5mm
Changed lines of the file:
@@
 F 0 "NT1" H 6500 2131 50  0000 C CNN
 F 1 "Net-Tie_2" H 6500 2040 50  0000 C CNN
-F 2 "NetTie:NetTie-2_THT_Pad1.0mm" H 6500 1950 50  0001 C CNN
+F 2 "NetTie:NetTie-2_SMD_Pad0.5mm" H 6500 1950 50  0001 C CNN
 F 3 "~" H 6500 1950 50  0001 C CNN
 	1    6500 1950
